Commit message: finished marble husky sensor config 5

File: submitted_models/marble_husky_sensor_config_5/urdf/robot_from_sdf.xacro (robot description, xacro)
@@ -1,5 +1,5 @@
 <?xml version='1.0' encoding='utf-8'?>
-<robot name='marble_husky_sensor_config_3' xmlns:xacro='http://ros.org/wiki/xacro'>
-  <xacro:arg name="name" default="marble_husky_sensor_config_3"/>
+<robot name='marble_husky_sensor_config_5' xmlns:xacro='http://ros.org/wiki/xacro'>
+  <xacro:arg name="name" default="marble_husky_sensor_config_5"/>
   <xacro:property name="robot_namespace" value="$(arg name)"/>
   <link name='${robot_namespace}/base_link'>
@@ -72,5 +72,5 @@
       <origin xyz='0 0 0' rpy='0 -0 0'/>
       <geometry>
-        <mesh filename='package://marble_husky_sensor_config_3/meshes/base_link.dae' scale='1 1 1'/>
+        <mesh filename='package://marble_husky_sensor_config_5/meshes/base_link.dae' scale='1 1 1'/>
       </geometry>
     </visual>
@@ -78,5 +78,5 @@
       <origin xyz='0.478 0 0.26' rpy='0 0.5236 0'/>
       <geometry>
-        <mesh filename='package://marble_husky_sensor_config_3/meshes/realsense.dae' scale='1 1 1'/>
+        <mesh filename='package://marble_husky_sensor_config_5/meshes/realsense.dae' scale='1 1 1'/>
       </geometry>
     </visual>
@@ -84,5 +84,5 @@
       <origin xyz='0.478 0 0.285' rpy='0 -0 0'/>
       <geometry>
-        <mesh filename='package://marble_husky_sensor_config_3/meshes/realsense.dae' scale='1 1 1'/>
+        <mesh filename='package://marble_husky_sensor_config_5/meshes/realsense.dae' scale='1 1 1'/>
       </geometry>
     </visual>
@@ -90,5 +90,5 @@
       <origin xyz='0.48 0 0.091' rpy='0 -0 0'/>
       <geometry>
-        <mesh filename='package://marble_husky_sensor_config_3/meshes/bumper.dae' scale='1 1 1'/>
+        <mesh filename='package://marble_husky_sensor_config_5/meshes/bumper.dae' scale='1 1 1'/>
       </geometry>
     </visual>
@@ -96,5 +96,5 @@
       <origin xyz='-0.48 0 0.091' rpy='0 -0 3.14159'/>
       <geometry>
-        <mesh filename='package://marble_husky_sensor_config_3/meshes/bumper.dae' scale='1 1 1'/>
+        <mesh filename='package://marble_husky_sensor_config_5/meshes/bumper.dae' scale='1 1 1'/>
       </geometry>
     </visual>
@@ -102,5 +102,5 @@
       <origin xyz='0 0 0' rpy='0 -0 0'/>
       <geometry>
-        <mesh filename='package://marble_husky_sensor_config_3/meshes/top_chassis.dae' scale='1 1 1'/>
+        <mesh filename='package://marble_husky_sensor_config_5/meshes/top_chassis.dae' scale='1 1 1'/>
       </geometry>
     </visual>
@@ -108,5 +108,5 @@
       <origin xyz='0.424 0 0.327' rpy='0 -0 0'/>
       <geometry>
-        <mesh filename='package://marble_husky_sensor_config_3/meshes/VLP16_base_1.dae' scale='1 1 1'/>
+        <mesh filename='package://marble_husky_sensor_config_5/meshes/VLP16_base_1.dae' scale='1 1 1'/>
       </geometry>
     </visual>
@@ -114,5 +114,5 @@
       <origin xyz='0.424 0 0.327' rpy='0 -0 0'/>
       <geometry>
-        <mesh filename='package://marble_husky_sensor_config_3/meshes/VLP16_base_2.dae' scale='1 1 1'/>
+        <mesh filename='package://marble_husky_sensor_config_5/meshes/VLP16_base_2.dae' scale='1 1 1'/>
       </geometry>
     </visual>
@@ -120,5 +120,5 @@
       <origin xyz='0.424 0 0.327' rpy='0 -0 0'/>
       <geometry>
-        <mesh filename='package://marble_husky_sensor_config_3/meshes/VLP16_scan.dae' scale='1 1 1'/>
+        <mesh filename='package://marble_husky_sensor_config_5/meshes/VLP16_scan.dae' scale='1 1 1'/>
       </geometry>
     </visual>
@@ -126,5 +126,5 @@
       <origin xyz='0.272 0 0.245' rpy='0 -0 0'/>
       <geometry>
-        <mesh filename='package://marble_husky_sensor_config_3/meshes/user_rail.dae' scale='1 1 1'/>
+        <mesh filename='package://marble_husky_sensor_config_5/meshes/user_rail.dae' scale='1 1 1'/>
       </geometry>
     </visual>
@@ -195,5 +195,5 @@
       <origin xyz='0 0 0' rpy='0 -0 0'/>
       <geometry>
-        <mesh filename='package://marble_husky_sensor_config_3/meshes/wheel.dae' scale='1 1 1'/>
+        <mesh filename='package://marble_husky_sensor_config_5/meshes/wheel.dae' scale='1 1 1'/>
       </geometry>
     </visual>
@@ -214,5 +214,5 @@
       <origin xyz='0 0 0' rpy='0 -0 0'/>
       <geometry>
-        <mesh filename='package://marble_husky_sensor_config_3/meshes/wheel.dae' scale='1 1 1'/>
+        <mesh filename='package://marble_husky_sensor_config_5/meshes/wheel.dae' scale='1 1 1'/>
       </geometry>
     </visual>
@@ -233,5 +233,5 @@
       <origin xyz='0 0 0' rpy='0 -0 0'/>
       <geometry>
-        <mesh filename='package://marble_husky_sensor_config_3/meshes/wheel.dae' scale='1 1 1'/>
+        <mesh filename='package://marble_husky_sensor_config_5/meshes/wheel.dae' scale='1 1 1'/>
       </geometry>
     </visual>
@@ -252,5 +252,5 @@
       <origin xyz='0 0 0' rpy='0 -0 0'/>
       <geometry>
-        <mesh filename='package://marble_husky_sensor_config_3/meshes/wheel.dae' scale='1 1 1'/>
+        <mesh filename='package://marble_husky_sensor_config_5/meshes/wheel.dae' scale='1 1 1'/>
       </geometry>
     </visual>
@@ -296,5 +296,5 @@
       <origin xyz='0 0 0.03' rpy='0 -0 0'/>
       <geometry>
-        <mesh filename='package://marble_husky_sensor_config_3/meshes/realsense.dae' scale='1 1 1'/>
+        <mesh filename='package://marble_husky_sensor_config_5/meshes/realsense.dae' scale='1 1 1'/>
       </geometry>
     </visual>

Commit message: Changed urdf/xacro file. Sensors seem to be floating?

File: submitted_models/marble_husky_sensor_config_5/urdf/robot_from_sdf.xacro (robot description, xacro)
@@ -27,10 +27,4 @@
       </geometry>
     </collision>
-    <collision name='base_link_fixed_joint_lump__camera/camera_link_collision_1'>
-      <origin xyz='0 0 0.05' rpy='0 -0 0'/>
-      <geometry>
-        <box size='0.0078 0.13 0.0192'/>
-      </geometry>
-    </collision>
     <collision name='base_link_fixed_joint_lump__camera/camera_link_collision_2'>
       <origin xyz='0.478 0 0.285' rpy='0 -0 0'/>
@@ -51,10 +45,4 @@
       </geometry>
     </collision>
-    <collision name='base_link_fixed_joint_lump__velodyne_gimbal_plate_base_link_collision_7'>
-      <origin xyz='0.424 0 0.4' rpy='0 -0 0'/>
-      <geometry>
-        <box size='0.1 0.1 0.01'/>
-      </geometry>
-    </collision>
     <collision name='base_link_fixed_joint_lump__sensor_tower_8'>
       <origin xyz='0.374 0 0.215' rpy='0 -0 0'/>
@@ -75,16 +63,4 @@
       </geometry>
     </visual>
-    <visual name='base_link_fixed_joint_lump__camera/camera_link_visual_1'>
-      <origin xyz='0.478 0 0.26' rpy='0 0.5236 0'/>
-      <geometry>
-        <mesh filename='package://marble_husky_sensor_config_5/meshes/realsense.dae' scale='1 1 1'/>
-      </geometry>
-    </visual>
-    <visual name='base_link_fixed_joint_lump__camera/camera_link_visual_2'>
-      <origin xyz='0.478 0 0.285' rpy='0 -0 0'/>
-      <geometry>
-        <mesh filename='package://marble_husky_sensor_config_5/meshes/realsense.dae' scale='1 1 1'/>
-      </geometry>
-    </visual>
     <visual name='base_link_fixed_joint_lump__front_bumper_link_visual_3'>
       <origin xyz='0.48 0 0.091' rpy='0 -0 0'/>
@@ -105,22 +81,4 @@
       </geometry>
     </visual>
-    <visual name='base_link_fixed_joint_lump__velodyne_base_link_visual_10'>
-      <origin xyz='0.424 0 0.327' rpy='0 -0 0'/>
-      <geometry>
-        <mesh filename='package://marble_husky_sensor_config_5/meshes/VLP16_base_1.dae' scale='1 1 1'/>
-      </geometry>
-    </visual>
-    <visual name='base_link_fixed_joint_lump__velodyne_base_link_visual_11'>
-      <origin xyz='0.424 0 0.327' rpy='0 -0 0'/>
-      <geometry>
-        <mesh filename='package://marble_husky_sensor_config_5/meshes/VLP16_base_2.dae' scale='1 1 1'/>
-      </geometry>
-    </visual>
-    <visual name='base_link_fixed_joint_lump__velodyne_visual_12'>
-      <origin xyz='0.424 0 0.327' rpy='0 -0 0'/>
-      <geometry>
-        <mesh filename='package://marble_husky_sensor_config_5/meshes/VLP16_scan.dae' scale='1 1 1'/>
-      </geometry>
-    </visual>
     <visual name='base_link_fixed_joint_lump__user_rail_link_visual_13'>
       <origin xyz='0.272 0 0.245' rpy='0 -0 0'/>
@@ -135,10 +93,4 @@
       </geometry>
     </visual>
-    <visual name='base_link_fixed_joint_lump__velodyne_gimbal_plate_15'>
-      <origin xyz='0.424 0 0.4' rpy='0 -0 0'/>
-      <geometry>
-        <box size='0.06 0.06 0.01'/>
-      </geometry>
-    </visual>
     <visual name='base_link_fixed_joint_lump__sensor_tower_16'>
       <origin xyz='0.374 0 0.215' rpy='0 -0 0'/>
@@ -154,29 +106,127 @@
     </visual>
   </link>
-  <sensor name='camera_front' update_rate='30'>
-    <parent link='${robot_namespace}/imu_link'/>
-    <origin xyz='0.468 0 0.36' rpy='0 -0 0'/>
-    <camera>
-      <image width='640' height='480' format='R8G8B8' hfov='1.5184' near='0.01' far='300' />
-    </camera>
-  </sensor>
-  <sensor name='camera_back' update_rate='30'>
-    <parent link='${robot_namespace}/base_link'/>
-    <origin xyz='0.468 0 0.36' rpy='0 -0 0'/>
-    <camera>
-      <image width='640' height='480' format='R8G8B8' hfov='1.5184' near='0.01' far='300' />
-    </camera>
-  </sensor>
-  <sensor name='planar_laser' update_rate='10'>
-    <parent link='${robot_namespace}/base_link'/>
-    <origin xyz='0.474 0 0.127' rpy='0 -0 0'/>
-  </sensor>
-  <sensor name='front_laser' update_rate='20'>
-    <parent link='${robot_namespace}/base_link'/>
-    <origin xyz='0.424 0 0.387' rpy='0 -0 0'/>
-  </sensor>
-  <sensor name='imu_sensor' update_rate='250'>
-    <parent link='${robot_namespace}/base_link'/>
-    <origin xyz='0.4379 0 0.52418' rpy='0 -0 0'/>
+  <sensor name='planar_laser' update_rate='20'>
+    <parent link='${robot_namespace}/base_link'/>
+    <origin xyz='0.485 0 0.166' rpy='0 -0 0'/>
+  </sensor>
+  <sensor name='camera_down' update_rate='15'>
+    <parent link='${robot_namespace}/base_link'/>
+    <origin xyz='0.44 0 0.41' rpy='0 0.5236 0'/>
+    <camera>
+      <image width='320' height='240' format='R8G8B8' hfov='1.5184' near='0.01' far='300' />
+    </camera>
+  </sensor>
+  <link name='${robot_namespace}/sensor_head_link'>
+    <inertial>
+      <origin xyz='0 0 0' rpy='0 -0 0'/>
+      <mass value='0.1'/>
+      <inertia ixx='0.01' ixy='0' ixz='0' iyy='0.01' iyz='0' izz='0.01'/>
+    </inertial>
+    <visual name='sensor_head_visual'>
+      <origin xyz='0 0 0' rpy='0 -0 0'/>
+      <geometry>
+        <box size='0.1 0.1 0.1'/>
+      </geometry>
+    </visual>
+    <visual name='base_link_fixed_joint_lump__velodyne_base_link_visual_10'>
+      <origin xyz='0 0 0.086' rpy='0 -0 0'/>
+      <geometry>
+        <mesh filename='package://marble_husky_sensor_config_5/meshes/VLP16_base_1.dae' scale='1 1 1'/>
+      </geometry>
+    </visual>
+    <visual name='base_link_fixed_joint_lump__velodyne_base_link_visual_11'>
+      <origin xyz='0 0 0.086' rpy='0 -0 0'/>
+      <geometry>
+        <mesh filename='package://marble_husky_sensor_config_5/meshes/VLP16_base_2.dae' scale='1 1 1'/>
+      </geometry>
+    </visual>
+    <visual name='base_link_fixed_joint_lump__velodyne_visual_12'>
+      <origin xyz='0 0 0.086' rpy='0 -0 0'/>
+      <geometry>
+        <mesh filename='package://marble_husky_sensor_config_5/meshes/VLP16_scan.dae' scale='1 1 1'/>
+      </geometry>
+    </visual>
+    <visual name='base_link_fixed_joint_lump__velodyne_base_link_visual_13'>
+      <origin xyz='0.12753 0 -0.076' rpy='3.14159 1.57079 -3e-06'/>
+      <geometry>
+        <mesh filename='package://marble_husky_sensor_config_5/meshes/VLP16_base_1.dae' scale='1 1 1'/>
+      </geometry>
+    </visual>
+    <visual name='base_link_fixed_joint_lump__velodyne_base_link_visual_14'>
+      <origin xyz='0.12753 0 -0.076' rpy='3.14159 1.57079 3.14159'/>
+      <geometry>
+        <mesh filename='package://marble_husky_sensor_config_5/meshes/VLP16_base_2.dae' scale='1 1 1'/>
+      </geometry>
+    </visual>
+    <visual name='base_link_fixed_joint_lump__velodyne_visual_15'>
+      <origin xyz='0.12753 0 -0.076' rpy='3.14159 1.57079 3.14159'/>
+      <geometry>
+        <mesh filename='package://marble_husky_sensor_config_5/meshes/VLP16_scan.dae' scale='1 1 1'/>
+      </geometry>
+    </visual>
+    <visual name='camera_front_visual'>
+      <origin xyz='0.158 0 0.0324' rpy='0 -0 0'/>
+      <geometry>
+        <box size='0.04 0.04 0.04'/>
+      </geometry>
+    </visual>
+    <visual name='camera_left_visual'>
+      <origin xyz='0 0.158 0.0324' rpy='0 -0 1.5708'/>
+      <geometry>
+        <box size='0.04 0.04 0.04'/>
+      </geometry>
+    </visual>
+    <visual name='camera_back_visual'>
+      <origin xyz='-0.158 0 0.0324' rpy='0 -0 0'/>
+      <geometry>
+        <box size='0.04 0.04 0.04'/>
+      </geometry>
+    </visual>
+    <visual name='camera_right_visual'>
+      <origin xyz='0 -0.158 0.0324' rpy='0 0 -1.5708'/>
+      <geometry>
+        <box size='0.04 0.04 0.04'/>
+      </geometry>
+    </visual>
+  </link>
+  <sensor name='imu_sensor' update_rate='50'>
+    <parent link='${robot_namespace}/sensor_head_link'/>
+    <origin xyz='0 0 0' rpy='0 -0 0'/>
+  </sensor>
+  <sensor name='horiz_laser' update_rate='20'>
+    <parent link='${robot_namespace}/sensor_head_link'/>
+    <origin xyz='0 0 0.086' rpy='0 -0 0'/>
+  </sensor>
+  <sensor name='vert_laser' update_rate='20'>
+    <parent link='${robot_namespace}/sensor_head_link'/>
+    <origin xyz='0.12753 0 -0.076' rpy='3.14159 1.57079 3.14159'/>
+  </sensor>
+  <sensor name='camera_front' update_rate='15'>
+    <parent link='${robot_namespace}/sensor_head_link'/>
+    <origin xyz='0.158 0 0.0324' rpy='0 -0 0'/>
+    <camera>
+      <image width='1280' height='960' format='R8G8B8' hfov='1.0472' near='0.01' far='300' />
+    </camera>
+  </sensor>
+  <sensor name='camera_left' update_rate='15'>
+    <parent link='${robot_namespace}/sensor_head_link'/>
+    <origin xyz='0 0.158 0.0324' rpy='0 -0 1.5708'/>
+    <camera>
+      <image width='1280' height='960' format='R8G8B8' hfov='1.0472' near='0.01' far='300' />
+    </camera>
+  </sensor>
+  <sensor name='camera_back' update_rate='15'>
+    <parent link='${robot_namespace}/sensor_head_link'/>
+    <origin xyz='-0.158 0 0.0324' rpy='0 -0 3.14159'/>
+    <camera>
+      <image width='1280' height='960' format='R8G8B8' hfov='1.0472' near='0.01' far='300' />
+    </camera>
+  </sensor>
+  <sensor name='camera_right' update_rate='15'>
+    <parent link='${robot_namespace}/sensor_head_link'/>
+    <origin xyz='0 -0.158 0.0324' rpy='0 0 -1.5708'/>
+    <camera>
+      <image width='1280' height='960' format='R8G8B8' hfov='1.0472' near='0.01' far='300' />
+    </camera>
   </sensor>
   <link name='${robot_namespace}/front_left_wheel_link'>
@@ -256,73 +306,11 @@
     </visual>
   </link>
-  <link name='${robot_namespace}/pan_gimbal_link'>
-    <inertial>
-      <origin xyz='0 0 0' rpy='0 -0 0'/>
-      <mass value='0.1'/>
-      <inertia ixx='1' ixy='0' ixz='0' iyy='1' iyz='0' izz='1'/>
-    </inertial>
-    <collision name='pan_gimbal_link_collision'>
-      <origin xyz='0 0 0' rpy='0 -0 0'/>
-      <geometry>
-        <cylinder radius='0.014' length='0.045'/>
-      </geometry>
-    </collision>
-    <visual name='pan_gimbal_link_visual'>
-      <origin xyz='0 0 0' rpy='0 -0 0'/>
-      <geometry>
-        <cylinder radius='0.014' length='0.045'/>
-      </geometry>
-    </visual>
-  </link>
-  <link name='${robot_namespace}/tilt_gimbal_link'>
-    <inertial>
-      <origin xyz='0 0 0' rpy='1.5708 -0 0'/>
-      <mass value='0.1'/>
-      <inertia ixx='1' ixy='0' ixz='0' iyy='1' iyz='0' izz='1'/>
-    </inertial>
-    <collision name='tilt_gimbal_link_collision'>
-      <origin xyz='0 0 0' rpy='1.5708 -0 0'/>
-      <geometry>
-        <cylinder radius='0.014' length='0.045'/>
-      </geometry>
-    </collision>
-    <visual name='tilt_gimbal_link_visual'>
-      <origin xyz='0 0 0' rpy='1.5708 -0 0'/>
-      <geometry>
-        <cylinder radius='0.014' length='0.045'/>
-      </geometry>
-    </visual>
-    <visual name='tilt_gimbal_link_fixed_joint_lump__camera/camera_link_visual_0'>
-      <origin xyz='0 0 0.03' rpy='0 -0 0'/>
-      <geometry>
-        <mesh filename='package://marble_husky_sensor_config_5/meshes/realsense.dae' scale='1 1 1'/>
-      </geometry>
-    </visual>
-    <visual name='tilt_gimbal_link_fixed_joint_lump_bot_camera_plate_link_visual_1'>
-      <origin xyz='0 0 0.017' rpy='0 -0 0'/>
-      <geometry>
-        <box size='0.025 0.13 0.007'/>
-      </geometry>
-    </visual>
-    <visual name='tilt_gimbal_link_fixed_joint_lump_bot_camera_plate_link_visual_2'>
-      <origin xyz='0 0 0.042' rpy='0 -0 0'/>
-      <geometry>
-        <box size='0.025 0.13 0.007'/>
-      </geometry>
-    </visual>
-    <visual name='flashlight_flashlight_light_source_lamp_viz_visual'>
-      <origin xyz='0 0 0.065' rpy='-0 1.3208 3.14'/>
-      <geometry>
-        <cylinder radius='0.019' length='0.005'/>
-      </geometry>
-    </visual>
-  </link>
-  <sensor name='camera_pan_tilt' update_rate='30'>
-    <parent link='${robot_namespace}/tilt_gimbal_link'/>
-    <origin xyz='0 0 0.03' rpy='0 -0 0'/>
-    <camera>
-      <image width='1280' height='720' format='R8G8B8' hfov='1.5184' near='0.01' far='300' />
-    </camera>
-  </sensor>
+  <joint name='sensor_head_joint' type='fixed'>
+    <origin xyz='0.4379 0 0.52418' rpy='0 -0 0'/>
+    <parent link='${robot_namespace}/base_link'/>
+    <child link='${robot_namespace}/sensor_head_link'/>
+    <axis xyz='0 0 1'/>
+    <limit lower='-1e+16' upper='1e+16' effort='-1' velocity='-1'/>
+  </joint>
   <joint name='front_left_wheel_joint' type='revolute'>
     <origin xyz='0.256 0.2854 0.03282' rpy='0 -0 0'/>
@@ -357,19 +345,3 @@
     <limit lower='-1e+16' upper='1e+16' effort='-1' velocity='-1'/>
   </joint>
-  <joint name='pan_gimbal_joint' type='revolute'>
-    <origin xyz='0.424 0 0.427' rpy='0 -0 0'/>
-    <parent link='${robot_namespace}/base_link'/>
-    <child link='${robot_namespace}/pan_gimbal_link'/>
-    <dynamics damping='0' friction='0' />
-    <axis xyz='0 0 1'/>
-    <limit lower='-1e+16' upper='1e+16' effort='-1' velocity='-1'/>
-  </joint>
-  <joint name='tilt_gimbal_joint' type='revolute'>
-    <origin xyz='0.424 0 0.46' rpy='0 -0 0'/>
-    <parent link='${robot_namespace}/pan_gimbal_link'/>
-    <child link='${robot_namespace}/tilt_gimbal_link'/>
-    <dynamics damping='0' friction='0' />
-    <axis xyz='0 1 0'/>
-    <limit lower='-2.79253' upper='2.79253' effort='-1' velocity='-1'/>
-  </joint>
 </robot>

Commit message: fixed imu frame

File: submitted_models/marble_husky_sensor_config_5/urdf/robot_from_sdf.xacro (robot description, xacro)
@@ -191,5 +191,5 @@
   </link>
   <sensor name='imu_sensor' update_rate='50'>
-    <parent link='${robot_namespace}/sensor_head_link'/>
+    <parent link='${robot_namespace}/base_link'/>
     <origin xyz='0 0 0' rpy='0 -0 0'/>
   </sensor>
